File: plexo-v-0-rev-a/plexo-v-0-rev-a.kicad_sch (KiCad schematic)
At the start: 9 parts, among them J2 Screw_Terminal_01x03, J3 Screw_Terminal_01x03, U1 74HC4051

Commit message: agregar sch
Parts:
- removed J2, J3: Screw_Terminal_01x03, symbol Connector:Screw_Terminal_01x03
- added C1, C2, C3, C4, C5, C6, C7: 100n, Capacitor_SMD:C_0805_2012Metric, symbol Device:C
- added J3: Screw_Terminal_01x06, Connector_PinSocket_2.54mm:PinSocket_1x06_P2.54mm_Vertical, symbol Connector:Screw_Terminal_01x06
- RV1, RV2, RV3, RV4, RV5, RV6: value R_Potentiometer -> 10k; footprint (none) -> Potentiometer_THT:Potentiometer_Alpha_RD901F-40-00D_Single_Vertical
- U1: LCSC (none) -> C9386
Connections:
- net +3V3: now also C7.1, J3.1 (Pin_1)
- net GND: now also C1.2, C2.2, C3.2, C4.2, C5.2, C6.2, C7.2, J3.3 (Pin_3)
- net pote3: now reaches RV3.2, U1.15 (A2)
- net pote3: now also C3.1
- net pote5: now reaches RV5.2, U1.1 (A4)
- net pote5: now also C5.1
- net at U1.3 (A): now also J3.2 (Pin_2)
- net pote1: now reaches RV1.2, U1.13 (A0)
- net pote1: now also C1.1
- net pote2: now reaches RV2.2, U1.14 (A1)
- net pote2: now also C2.1
- net at U1.10 (S1): now also J3.5 (Pin_5)
- net at U1.11 (S0): now also J3.4 (Pin_4)
- net pote4: now reaches RV4.2, U1.12 (A3)
- net pote4: now also C4.1
- net pote6: now reaches RV6.2, U1.5 (A5)
- net pote6: now also C6.1
- net at U1.9 (S2): now also J3.6 (Pin_6)
Other:
- moved on the sheet: RV1, RV2, U1

Commit message: agregar plexo-v-0
Parts:
- added H1, H2: MountingHole, MountingHole:MountingHole_3.2mm_M3, symbol Mechanical:MountingHole
Connections:
- net sel0: now reaches J3.4 (Pin_4), U1.11 (S0)
- net sel1: now reaches J3.5 (Pin_5), U1.10 (S1)
- net sel2: now reaches J3.6 (Pin_6), U1.9 (S2)
Changed lines of the file:
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@@
+		)
+	)
+	(label "sel0"
+		(at 46.99 58.42 0)
+		(effects
+			(font
+				(size 1.27 1.27)
+			)
+			(justify left bottom)
 		)
 	)
@@
 		)
 	)
+	(label "sel1"
+		(at 46.99 60.96 0)
+		(effects
+			(font
+				(size 1.27 1.27)
+			)
+			(justify left bottom)
+		)
+	)
 	(label "pote1"
 		(at 115.57 31.75 180)
@@
 			)
 			(justify right bottom)
+		)
+	)
+	(label "sel2"
+		(at 46.99 63.5 0)
+		(effects
+			(font
+				(size 1.27 1.27)
+			)
+			(justify left bottom)
 		)
 	)
@@
 	)
 	(symbol
+		(lib_id "Mechanical:MountingHole")
+		(at 119.38 87.63 0)
+		(unit 1)
+		(body_style 1)
+		(exclude_from_sim no)
+		(in_bom no)
+		(on_board yes)
+		(in_pos_files yes)
+		(dnp no)
+		(fields_autoplaced yes)
+		(property "Reference" "H1"
+			(at 121.92 86.3599 0)
+			(show_name no)
+			(do_not_autoplace no)
+			(effects
+				(font
+					(size 1.27 1.27)
+				)
+				(justify left)
+			)
+		)
+		(property "Value" "MountingHole"
+			(at 121.92 88.8999 0)
+			(show_name no)
+			(do_not_autoplace no)
+			(effects
+				(font
+					(size 1.27 1.27)
+				)
+				(justify left)
+			)
+		)
+		(property "Footprint" "MountingHole:MountingHole_3.2mm_M3"
+			(at 119.38 87.63 0)
+			(hide yes)
+			(show_name no)
+			(do_not_autoplace no)
+			(effects
+				(font
+					(size 1.27 1.27)
+				)
+			)
+		)
+		(property "Datasheet" ""
+			(at 119.38 87.63 0)
+			(hide yes)
+			(show_name no)
+			(do_not_autoplace no)
+			(effects
+				(font
+					(size 1.27 1.27)
+				)
+			)
+		)
+		(property "Description" "Mounting Hole without connection"
+			(at 119.38 87.63 0)
+			(hide yes)
+			(show_name no)
+			(do_not_autoplace no)
+			(effects
+				(font
+					(size 1.27 1.27)
+				)
+			)
+		)
+		(instances
+			(project "plexo-v-0-rev-a"
+				(path "/d5260b14-2c1b-40b1-b976-e20b39ad53be"
+					(reference "H1")
+					(unit 1)
+				)
+			)
+		)
+	)
+	(symbol
 		(lib_id "Device:R_Potentiometer")
 		(at 184.15 30.48 180)
@@
 					(unit 1)
 				)
+			)
+		)
+	)
+	(symbol
+		(lib_id "Mechanical:MountingHole")
+		(at 140.97 87.63 0)
+		(unit 1)
+		(body_style 1)
+		(exclude_from_sim no)
+		(in_bom no)
+		(on_board yes)
+		(in_pos_files yes)
+		(dnp no)
+		(fields_autoplaced yes)
+		(property "Reference" "H2"
+			(at 143.51 86.3599 0)
+			(show_name no)
+			(do_not_autoplace no)
+			(effects
+				(font
+					(size 1.27 1.27)
+				)
+				(justify left)
+			)
+		)
+		(property "Value" "MountingHole"
+			(at 143.51 88.8999 0)
+			(show_name no)
+			(do_not_autoplace no)
+			(effects
+				(font
+					(size 1.27 1.27)
+				)
+				(justify left)
+			)
+		)
+		(property "Footprint" "MountingHole:MountingHole_3.2mm_M3"
+			(at 140.97 87.63 0)
+			(hide yes)
+			(show_name no)
+			(do_not_autoplace no)
+			(effects
+				(font
+					(size 1.27 1.27)
+				)
+			)
+		)
+		(property "Datasheet" ""
+			(at 140.97 87.63 0)
+			(hide yes)
+			(show_name no)
+			(do_not_autoplace no)
+			(effects
+				(font
+					(size 1.27 1.27)
+				)
+			)
+		)
+		(property "Description" "Mounting Hole without connection"
+			(at 140.97 87.63 0)
+			(hide yes)
+			(show_name no)
+			(do_not_autoplace no)
+			(effects
+				(font
+					(size 1.27 1.27)
+				)
+			)
+		)
+		(instances
+			(project "plexo-v-0-rev-a"
+				(path "/d5260b14-2c1b-40b1-b976-e20b39ad53be"
+					(reference "H2")
+					(unit 1)
+				)
